Commit message: remake object size and add some code to script

File: env_urdf/objects/obj_2.urdf.xacro (robot description, xacro)
@@ -21,7 +21,7 @@
   </link>
   <gazebo reference="base_link">
-    <material>Gazebo/Blue</material>
-    <!--mu1>0.4</mu1>
-    <mu2>0.4</mu2-->
+    <material>Gazebo/Green</material>
+    <mu1>0.4</mu1>
+    <mu2>0.4</mu2>
   </gazebo>
 </robot>

File: env_urdf/objects/obj_3.urdf.xacro (robot description, xacro)
@@ -21,7 +21,7 @@
   </link>
   <gazebo reference="base_link">
-    <material>Gazebo/Blue</material>
-    <!--mu1>0.4</mu1>
-    <mu2>0.4</mu2-->
+    <material>Gazebo/Yellow</material>
+    <mu1>0.4</mu1>
+    <mu2>0.4</mu2>
   </gazebo>
 </robot>

File: env_urdf/table.urdf.xacro (robot description, xacro)
@@ -30,4 +30,6 @@
   <gazebo reference="base_link">
     <material>Gazebo/DarkGrey</material>
+    <mu1>0.4</mu1>
+    <mu2>0.4</mu2>
   </gazebo>
   <xacro:camera_gazebo_v0/>
