Commit message: some script change

File: env_urdf/camera.urdf.xacro (robot description, xacro)
@@ -13,6 +13,6 @@
           <box size="0.05 0.05 0.05"/>
         </geometry>
-        <origin xyz="0 0 1" rpy="0 0 0"/>
-        <material name="red"/>
+	  <origin xyz="0.25 0 0.36" rpy="0 ${PI*6/25} ${PI}"/>
+        <!--material name="red"/-->
       </visual>
       <!--collision>

File: env_urdf/objects/camera.gazebo.xacro (robot description, xacro)
@@ -3,9 +3,9 @@
   <xacro:include filename="$(find ur5_gripper_moveit_config)/env_urdf/common.xacro"/>
   <xacro:macro name="camera_gazebo_v0">
-    <gazebo reference="camera_link">
+    <gazebo reference="base_link">
       <sensor type="camera" name="camera_sensor">
         <update_rate>10.0</update_rate>
-        <camera name="bird_view">
-		<pose>0.25 0 0.36 0 ${PI*6/25} ${PI}</pose>
+        <camera name="obj_camera">
+		<pose>0 0 0 0 0 0</pose>
           <horizontal_fov>1.3962634</horizontal_fov>
           <image>
@@ -27,5 +27,5 @@
           <alwaysOn>true</alwaysOn>
           <updateRate>0.0</updateRate>
-          <cameraName>camera</cameraName>
+          <cameraName>obj_camera</cameraName>
           <imageTopicName>image_raw</imageTopicName>
           <cameraInfoTopicName>camera_info</cameraInfoTopicName>

File: env_urdf/objects/obj_2.urdf.xacro (robot description, xacro)
@@ -2,4 +2,5 @@
 <robot name="obj_1" xmlns:xacro="http://ros.org/wiki/xacro">
   <xacro:include filename="$(find ur5_gripper_moveit_config)/env_urdf/common.xacro"/>
+  <xacro:include filename="$(find ur5_gripper_moveit_config)/env_urdf/objects/camera.gazebo.xacro"/>
   <link name="base_link">
     <inertial>
@@ -25,3 +26,4 @@
     <mu2>0.4</mu2>
   </gazebo>
+  <xacro:camera_gazebo_v0/>
 </robot>
