Commit message: change table size and related variable

File: env_urdf/table.urdf.xacro (robot description, xacro)
@@ -12,10 +12,10 @@
     <inertial>
       <origin xyz="0 0 0" rpy="0 0 0"/>
-      <box_inertial mass="1.0" height="0.8" width="0.8" depth="0.3"/>
+      <box_inertial mass="1.0" height="0.4" width="0.4" depth="0.3"/>
     </inertial>
     <visual>
       <origin xyz="0 0 0" rpy="0 0 0"/>
       <geometry>
-        <box size="0.8 0.8 0.3"/>
+        <box size="0.4 0.4 0.3"/>
       </geometry>
     </visual>
@@ -23,5 +23,5 @@
       <origin xyz="0 0 0" rpy="0 0 0"/>
       <geometry>
-        <box size="0.8 0.8 0.3" />
+        <box size="0.4 0.4 0.3" />
       </geometry>
     </collision>

Commit message: add some script

File: env_urdf/table.urdf.xacro (robot description, xacro)
@@ -12,10 +12,10 @@
     <inertial>
       <origin xyz="0 0 0" rpy="0 0 0"/>
-      <box_inertial mass="1.0" height="0.4" width="0.4" depth="0.3"/>
+      <box_inertial mass="1.0" height="0.3" width="0.3" depth="0.3"/>
     </inertial>
     <visual>
       <origin xyz="0 0 0" rpy="0 0 0"/>
       <geometry>
-        <box size="0.4 0.4 0.3"/>
+        <box size="0.3 0.3 0.3"/>
       </geometry>
     </visual>
@@ -23,5 +23,5 @@
       <origin xyz="0 0 0" rpy="0 0 0"/>
       <geometry>
-        <box size="0.4 0.4 0.3" />
+        <box size="0.3 0.3 0.3" />
       </geometry>
     </collision>

Commit message: add pan and some change for it

File: env_urdf/table.urdf.xacro (robot description, xacro)
@@ -29,5 +29,5 @@
   <xacro:bird_camera_v0 parent="base_link"/>
   <gazebo reference="base_link">
-    <material>Gazebo/DarkGrey</material>
+    <material>Gazebo/Grey</material>
     <mu1>0.4</mu1>
     <mu2>0.4</mu2>
